File: Software/rele-wifi-villalbayrojas/rele-wifi-villalbayrojas.kicad_sch (KiCad schematic)
At the start: 31 parts, among them K5 G5V-2, K6 G5V-2, K7 G5V-2, K8 G5V-2, Q4 Q_NPN, Q5 Q_NPN, Q6 Q_NPN, Q7 Q_NPN, U1 AMS1117-3.3, U4 PC817, U5 PC817, U6 PC817, U7 PC817

Commit message: Subi o nuevo
Parts:
- added C3, C4, C5, C6, C7: C, symbol Device:C
- added J1: Relay1, symbol Connector:Screw_Terminal_01x03
- added J2: Relay2, symbol Connector:Screw_Terminal_01x03
- added J3: Relay3, symbol Connector:Screw_Terminal_01x03
- added J4: Relay4, symbol Connector:Screw_Terminal_01x03
- added R1: R, symbol Device:R
- added SW1, SW2: SW_MEC_5G, symbol Switch:SW_MEC_5G
- added U2: ESP32-WROOM-32, RF_Module:ESP32-WROOM-32, symbol RF_Module:ESP32-WROOM-32
- K5, K6, K7, K8: footprint Relay_THT:Relay_DPDT_Omron_G5V-2 -> Relay_THT:Relay_DPDT_Finder_30.22
Connections:
- net +3.3V: now also C3.1, C4.1, R1.1, U2.2 (VDD)
- net GND: now also C3.2, C4.2, C5.2, C6.2, C7.2, SW1.1 (A), SW1.2 (A), SW2.1 (A), SW2.2 (A), U2.1 (GND), U2.15 (GND), U2.38 (GND), U2.39 (GND)
- net IO_18: now reaches D13.1 (K)
- net IO_18: now also U2.30 (IO18)
- net at Q5.B, R10.2: no longer R10.1, U5.3
- net at Q6.B, R12.2: no longer R12.1, U6.3
- net at R8.1, U4.3: no longer Q4.B, R8.2
- net at Q7.B, R14.2: no longer R14.1, U7.3
- net IO_19: now reaches D9.1 (K)
- net IO_19: now also U2.31 (IO19)
- net NC-1.1: now reaches K5.11
- net NC-1.1: now also K6.11, K7.11, K8.11
- net COM-1.1: now reaches K5.13
- net COM-1: now reaches K5.4
- net COM-1: now also J1.2 (Pin_2)
- net NC-1: now reaches K5.6
- net NC-1: now also K6.6, K7.6, K8.6, J1.3 (Pin_3)
- net NO-1: now reaches K5.8
- net NO-1: now also K6.8, K7.8, K8.8, J1.1 (Pin_1)
- net NO-1.1: now reaches K5.9
- net NO-1.1: now also K6.9, K7.9, K8.9
- net IO_21: now reaches D7.1 (K)
- net IO_21: now also U2.33 (IO21)
- net COM-4.1: now reaches K8.13
- net COM-4: now reaches K8.4
- net COM-4: now also J4.2 (Pin_2)
- net COM-3.1: now reaches K6.13
- net COM-3: now reaches K6.4
- net COM-3: now also J3.2 (Pin_2)
- net COM-2.1: now reaches K7.13
- net COM-2: now reaches K7.4
- net COM-2: now also J2.2 (Pin_2)
- net IO_5: now reaches D11.1 (K)
- net IO_5: now also U2.29 (IO5)
- new net: R12.1, U6.3
- new net: Q4.B, R8.2
- new net: R14.1, U7.3
- new net: R10.1, U5.3
- new net IO_0: C7.1, SW2.3 (B), SW2.4 (B), U2.25 (IO0)
- new net NC-2: J2.3 (Pin_3)
- new net NC-3: J3.3 (Pin_3)
- new net NC-4: J4.3 (Pin_3)
- new net NO-2: J2.1 (Pin_1)
- new net NO-3: J3.1 (Pin_1)
- new net NO-4: J4.1 (Pin_1)
- new net RESET: C5.1, C6.1, R1.2, SW1.3 (B), SW1.4 (B), U2.3 (EN)
- new net RX: U2.35 (TXD0/IO1)
- new net TX: U2.34 (RXD0/IO3)
Other:
- moved on the sheet: C1, C2, U1
